Commit message: No code changes made

File: cart_pole.urdf (robot description, URDF)
Before this commit: robot cart_pole, 2 links, 1 joints
Links:
- link pole_link: geometry collision cylinder length=0.45 radius=0.01; visual cylinder length=0.45 radius=0.01
Joints:
- removed joint pivot_joint
- added joint pole_joint: type revolute, parent cart_link, child pole_link, origin xyz=0 0 0.2 rpy=0 0 0, axis 0 1 0, limit lower=-3.14 upper=3.14 effort=100 velocity=50
