Commit message: Refine URDF model for flagpole: improve comments, adjust mass and dimensions for stability

File: flagpole.urdf (robot description, URDF)
Before this commit: robot flagpole, 6 links, 5 joints
Links:
- link bl_wheel_1: geometry collision cylinder length=0.02 radius=0.07; visual cylinder length=0.02 radius=0.07
- link br_wheel_1: geometry collision cylinder length=0.02 radius=0.07; visual cylinder length=0.02 radius=0.07
- link pole_1: geometry collision cylinder length=0.5 radius=0.03; collision sphere radius=0.06
- link tl_wheel_1: geometry collision cylinder length=0.02 radius=0.07; visual cylinder length=0.02 radius=0.07
- link tr_wheel_1: geometry collision cylinder length=0.02 radius=0.07; visual cylinder length=0.02 radius=0.07

Commit message: Implement PID control for cart-pole simulation and enhance URDF model with improved comments and friction settings

File: flagpole.urdf (robot description, URDF)
Before this commit: robot flagpole, 6 links, 5 joints
Links:
- link bl_wheel_1: mass 1.0 -> None; geometry 
- link br_wheel_1: mass 1.0 -> None; geometry 
- link tr_wheel_1: mass 1.0 -> None; geometry 

File: flagpole_decoupled.urdf (robot description, URDF)
Before this commit: robot flagpole_decoupled, 6 links, 5 joints
Links:
- removed link base_link
- removed link rod_link
- removed link wheel_1
- removed link wheel_2
- removed link wheel_3
- removed link wheel_4
- added link cart, mass 10.0; collision box size=0.5 0.3 0.1; visual box size=0.5 0.3 0.1
- added link pole, mass 1.0; collision cylinder length=0.6 radius=0.03; collision sphere radius=0.06
- added link wheel_fl; visual cylinder length=0.05 radius=0.08
- added link wheel_fr; visual cylinder length=0.05 radius=0.08
- added link wheel_rl; visual cylinder length=0.05 radius=0.08
- added link wheel_rr; visual cylinder length=0.05 radius=0.08
Joints:
- removed joint rod_base_joint
- removed joint wheel_1_joint
- removed joint wheel_2_joint
- removed joint wheel_3_joint
- removed joint wheel_4_joint
- added joint pole_joint: type revolute, parent cart, child pole, origin xyz=0 0 0.1 rpy=0 0 0, axis 0 1 0, limit lower=-0.87266 upper=0.87266 effort=50 velocity=2
- added joint wheel_fl_joint: type fixed, parent cart, child wheel_fl, origin xyz=0 0 0 rpy=0 0 0
- added joint wheel_fr_joint: type fixed, parent cart, child wheel_fr, origin xyz=0 0 0 rpy=0 0 0
- added joint wheel_rl_joint: type fixed, parent cart, child wheel_rl, origin xyz=0 0 0 rpy=0 0 0
- added joint wheel_rr_joint: type fixed, parent cart, child wheel_rr, origin xyz=0 0 0 rpy=0 0 0

Commit message: Refine URDF model for flagpole: enhance comments for clarity and detail on components

File: flagpole.urdf (robot description, URDF)
Before this commit: robot flagpole, 6 links, 5 joints
Links:
- link bl_wheel_1: mass None -> 1.0; geometry collision cylinder length=0.02 radius=0.07; visual cylinder length=0.02 radius=0.07
- link br_wheel_1: mass None -> 1.0; geometry collision cylinder length=0.02 radius=0.07; visual cylinder length=0.02 radius=0.07
- link tr_wheel_1: mass None -> 1.0; geometry collision cylinder length=0.02 radius=0.07; visual cylinder length=0.02 radius=0.07
